File: Timers.kicad_sch (KiCad schematic)
At the start: 4 parts, among them U13 4040, U14 4040, U15 4040, U6 4011

Commit message: Complete new version
Signed-off-by: Oliver Gaskell <og305@cam.ac.uk>
Parts:
- removed U6: 4011, Package_DIP:DIP-14_W7.62mm_Socket, symbol 4xxx:4011
- added TP6, TP7: TestPoint, TestPoint:TestPoint_Pad_D2.0mm, symbol Connector:TestPoint
Connections:
- net 4096CLK: now also TP6.1
- net 16s_Timer: now reaches U15.1 (Q11)
- net 128CLK: now reaches U13.13 (Q7)
- net 128CLK: now also U15.10 (CLK), TP7.1
- net 256CLK: no longer names the net of U13.4 (Q6)
- net 256CLK: no longer U15.10 (CLK)
- no-connect marks 31 -> 32
