File: state_machine.kicad_sch (KiCad schematic)
At the start: 15 parts, among them U1 4011, U11 4012, U12 74LS573, U3 4011, U4 4011, U5 4011, U6 4011, U7 4011, U8 4011

Commit message: Complete new version
Signed-off-by: Oliver Gaskell <og305@cam.ac.uk>
Parts:
- removed U8: 4011, Package_DIP:DIP-14_W7.62mm_Socket, symbol 4xxx:4011
- added unit 3 of U6
- added unit 4 of U6
- D6, D7: footprint LED_THT:LED_D5.0mm -> LED_SMD:LED_0603_1608Metric_Pad1.05x0.95mm_HandSolder
- R10, R9: value 220R -> 180; footprint Resistor_THT:R_Axial_DIN0207_L6.3mm_D2.5mm_P7.62mm_Horizontal -> Resistor_SMD:R_0603_1608Metric_Pad0.98x0.95mm_HandSolder
- TP3, TP4: footprint TestPoint:TestPoint_THTPad_D3.0mm_Drill1.5mm -> TestPoint:TestPoint_Pad_D2.0mm
Connections:
- net SM_Ok: now also U3.8, U3.9; no longer U3.1, U3.2
- net Timers/Reset_Counting: now also U3.11; no longer U3.10
- net at U7.10, U7.12: now also U6.8
- net at U7.3, U7.5: now also U6.12
- net at U3.6: now also U3.3; no longer U3.11
- net at U3.12, U3.13: now also U3.4; no longer U1.11
- net at U3.5: now also U3.10; no longer U3.3
- net at U12.3 (D1): now also U6.11
- net at U11.13: now also U6.9
- new net: U6.10, U6.13
- new net: U1.11, U3.1, U3.2
Other:
- sheet Timers ports: added 16s_Timer; removed 10s_Timer
- moved on the sheet: U3A, U3C, U3D, U7A, U7C, U7D
