File: trig_plugdet.kicad_sch (KiCad schematic)
At the start: 16 parts, among them U1 4011, U9 LM2901

Commit message: Complete new version
Signed-off-by: Oliver Gaskell <og305@cam.ac.uk>
Parts:
- D2, D5: footprint LED_THT:LED_D5.0mm -> LED_SMD:LED_0603_1608Metric_Pad1.05x0.95mm_HandSolder
- D3: renamed from D4; footprint LED_THT:LED_D5.0mm -> LED_SMD:LED_0603_1608Metric_Pad1.05x0.95mm_HandSolder
- D4: renamed from D3; footprint LED_THT:LED_D5.0mm -> LED_SMD:LED_0603_1608Metric_Pad1.05x0.95mm_HandSolder
- R4, R7: value 220R -> 180; footprint Resistor_THT:R_Axial_DIN0207_L6.3mm_D2.5mm_P7.62mm_Horizontal -> Resistor_SMD:R_0603_1608Metric_Pad0.98x0.95mm_HandSolder
- R5: renamed from R6; value 220R -> 180; footprint Resistor_THT:R_Axial_DIN0207_L6.3mm_D2.5mm_P7.62mm_Horizontal -> Resistor_SMD:R_0603_1608Metric_Pad0.98x0.95mm_HandSolder
- R6: renamed from R5; value 220R -> 180; footprint Resistor_THT:R_Axial_DIN0207_L6.3mm_D2.5mm_P7.62mm_Horizontal -> Resistor_SMD:R_0603_1608Metric_Pad0.98x0.95mm_HandSolder
- U9: value LM2901 -> TLC3704
Connections:
- net BPS_Trig: now also JP3.2 (C); no longer JP3.3 (B), U1.3
- net TPS_Trig: now also JP4.2 (C); no longer JP4.3 (B), U1.4
- net at U1.5, U1.6: now also JP4.3 (B), U9.1; no longer JP4.1 (A)
- net at U1.1, U1.2: now also JP3.3 (B), U9.2; no longer JP3.1 (A)
- new net: JP4.1 (A), U1.4
- new net: JP3.1 (A), U1.3
Other:
- moved on the sheet: D4, D5, JP3, JP4, R6, R7, RV1, RV3, U1A, U1B
